File: elec/layout/default/esp32-s3.kicad_pcb (KiCad board)
At the start: 2 copper layers, 225.7 x 100.8 mm, 0 parts

Commit message: initial design
Parts:
- added C1: 100.0 nF, lib:C0402, F.Cu at (164.6, 121.9)
- added C2: 10.0 uF, lib:C0805, F.Cu at (167.2, 112.1)
- added C3: 10.0 uF, lib:C0805, F.Cu at (159.0, 118.5)
- added R1: 8.2 KΩ, lib:R0402, F.Cu at (164.6, 117.9)
- added U1: , lib:WIRELM-SMD_ESP32-S3-WROOM-1, F.Cu at (160.2, 94.0)
- added U2: , lib:KEY-SMD_4P-L4.2-W3.2-P2.20-LS4.6, F.Cu at (159.9, 112.8)
Other:
- board size 225.7 x 100.8 mm -> 66.4 x 94.6 mm
