File: elec/layout/default/esp32-s3.kicad_pcb (KiCad board)
At the start: 2 copper layers, 6 parts

Commit message: Fix and relink layouts. Apply v0.3 updates
Connections:
- net RXD0 renamed rxd0
- net TXD0 renamed txd0
- net cs renamed io10
- net dm renamed io19
- net dp renamed io20
- net gnd renamed ic-gnd
- net hv renamed vcc
- net in renamed en
- net miso renamed io13
- net mosi renamed io11
- net sck renamed io12
- net scl renamed io6
- net sda renamed io7
- net tck renamed io39
- net tdi renamed io41
- net tdo renamed io40
- net tms renamed io42
