File: elec/layout/default/esp32-s3.kicad_pcb (KiCad board)
At the start: 2 copper layers, 6 parts

Commit message: build with latest
Connections:
- net en renamed in
- net ic-gnd renamed gnd
- net rxd0 renamed RXD0
- net txd0 renamed TXD0
- net vcc renamed hv
