File: elec/layout/base/base.kicad_pcb (KiCad board)
At the start: 2 copper layers, 38 parts

Commit message: Fix and relink layouts. Apply v0.3 updates
Parts:
- removed U10: , lib:IND-SMD_L2.5-W2.0_WPN252012H
- removed U11: , lib:LED0603-RD
- removed U12: , lib:KEY-SMD_4P-L4.2-W3.2-P2.20-LS4.6
- added L1: 1.5µH ±20%, lib:IND-SMD_L2.5-W2.0_WPN252012H, F.Cu at (217.7, 119.6)
- added L2: 1.5µH ±20%, lib:IND-SMD_L2.5-W2.0_WPN252012H, F.Cu at (210.7, 138.6)
- added LED1: 2V, lib:LED0603-RD, F.Cu at (208.9, 135.2)
- R10, R5, R8: value 10kΩ ±1% 62.5mW -> 1kΩ ±1% 62.5mW
- R4, R7: value 10kΩ ±1% 62.5mW -> infΩ infW
- U2: footprint lib:IND-SMD_L2.5-W2.0_WPN252012H -> lib:KEY-SMD_4P-L4.2-W3.2-P2.20-LS4.6
Connections:
- net A5 renamed cc1
- net A8 renamed sub1
- net B5 renamed cc2
- net B8 renamed sub2
- net CD renamed cd
- net DAT1_RSV_ renamed dat1_rsv_
- net DAT2_RSV_ renamed dat2_rsv_
- net EN renamed _3v3_reg.ic-vina
- net RXD0 renamed rxd0
- net TXD0 renamed txd0
- net VBUS renamed usb_conn-vcc
- net VINA renamed _5v_reg.ic-vina
- net _3v3_reg-PG renamed _3v3_reg.ic-pg
- net _3v3_reg-out renamed _3v3_reg.feedback_div-out
- net _5v_reg-L1 renamed _5v_reg.ic-l1
- net _5v_reg-L2 renamed _5v_reg.ic-l2
- net _5v_reg-PG renamed _5v_reg.ic-pg
- net _5v_reg-out renamed _5v_reg.feedback_div-out
- net dm renamed usb-
- net dp renamed usb+
- net hv renamed _5v_reg-vcc
- net hv-2 renamed vcc
- net io renamed io1
- C1 pad 1: hv-1 -> uc.ic-vcc
- C1 pad 2: gnd -> uc.ic-gnd
- C10 pad 2: gnd -> uc.ic-gnd
- C11 pad 1: hv-1 -> uc.ic-vcc
- C11 pad 2: gnd -> uc.ic-gnd
- C12 pad 1: hv-1 -> uc.ic-vcc
- C12 pad 2: gnd -> uc.ic-gnd
- C13 pad 2: gnd -> uc.ic-gnd
- C14 pad 1: hv-1 -> uc.ic-vcc
- C14 pad 2: gnd -> uc.ic-gnd
- C2 pad 1: hv-1 -> uc.ic-vcc
- C2 pad 2: gnd -> uc.ic-gnd
- C3 pad 1: hv-1 -> uc.ic-vcc
- C3 pad 2: gnd -> uc.ic-gnd
- C4 pad 2: gnd -> uc.ic-gnd
- C5 pad 2: gnd -> uc.ic-gnd
- C6 pad 2: gnd -> uc.ic-gnd
- C7 pad 2: gnd -> uc.ic-gnd
- C8 pad 2: gnd -> uc.ic-gnd
- C9 pad 2: gnd -> uc.ic-gnd
- R1 pad 1: hv-1 -> uc.ic-vcc
- R1 pad 2: in -> en
- R10 pad 2: gnd -> uc.ic-gnd
- R11 pad 2: hv-1 -> uc.ic-vcc
- R12 pad 2: hv-1 -> uc.ic-vcc
- R2 pad 2: gnd -> uc.ic-gnd
- R3 pad 2: gnd -> uc.ic-gnd
- R5 pad 2: gnd -> uc.ic-gnd
- R6 pad 2: gnd -> uc.ic-gnd
- R7 pad 1: hv-1 -> uc.ic-vcc
- R8 pad 2: gnd -> uc.ic-gnd
- R9 pad 2: gnd -> uc.ic-gnd
- U1 pad 1: gnd -> uc.ic-gnd
- U1 pad 2: hv-1 -> uc.ic-vcc
- U1 pad 3: in -> en
- U1 pad 40: gnd -> uc.ic-gnd
- U1 pad 41: gnd -> uc.ic-gnd
- U2 pad 1: _3v3_reg-L1 -> en
- U2 pad 2: _3v3_reg-L2 -> en
- U3 pad 1: (no net) -> uc.ic-vcc
- U3 pad 3: (no net) -> uc.ic-gnd
- U3 pad 5: (no net) -> uc.ic-gnd
- U3 pad 7: (no net) -> _7
- U3 pad 9: (no net) -> uc.ic-gnd
- U4 pad 1: gnd -> uc.ic-gnd
- U4 pad 2: gnd -> uc.ic-gnd
- U4 pad 3: gnd -> uc.ic-gnd
- U4 pad 4: gnd -> uc.ic-gnd
- U4 pad A1: gnd -> uc.ic-gnd
- U4 pad A12: gnd -> uc.ic-gnd
- U4 pad B1: gnd -> uc.ic-gnd
- U4 pad B12: gnd -> uc.ic-gnd
- U5 pad 13: gnd -> uc.ic-gnd
- U5 pad 15: gnd -> uc.ic-gnd
- U5 pad 2: gnd -> uc.ic-gnd
- U6 pad 13: gnd -> uc.ic-gnd
- U6 pad 15: gnd -> uc.ic-gnd
- U6 pad 2: gnd -> uc.ic-gnd
- U6 pad 4: hv-1 -> uc.ic-vcc
- U6 pad 5: hv-1 -> uc.ic-vcc
- U6 pad 6: _3v3_reg-L2 -> _3v3_reg.ic-l2
- U6 pad 7: _3v3_reg-L2 -> _3v3_reg.ic-l2
- U6 pad 8: _3v3_reg-L1 -> _3v3_reg.ic-l1
- U6 pad 9: _3v3_reg-L1 -> _3v3_reg.ic-l1
- U7 pad 10: gnd -> uc.ic-gnd
- U7 pad 11: gnd -> uc.ic-gnd
- U7 pad 12: gnd -> uc.ic-gnd
- U7 pad 13: gnd -> uc.ic-gnd
- U7 pad 4: hv-1 -> uc.ic-vcc
- U7 pad 6: gnd -> uc.ic-gnd
- U8 pad 1: hv-1 -> uc.ic-vcc
- U8 pad 3: gnd -> uc.ic-gnd
- U9 pad 1: gnd -> uc.ic-gnd
- U9 pad 2: hv-1 -> uc.ic-vcc
Routing:
- net (no net): track 230.4 -> 0.00 mm, vias 8 -> 0
- net uc.ic-vcc: track 0.00 -> 91.0 mm, vias 0 -> 2
- net vcc: track 0.00 -> 42.3 mm, vias 0 -> 2
- net uc.ic-gnd: track 0.00 -> 28.1 mm, vias 0 -> 2
- net _3v3_reg.ic-vina: track 0.00 -> 19.5 mm, vias 0 -> 2
- net scl: track 0.00 -> 15.3 mm
- net sda: track 0.00 -> 9.46 mm
- net en: track 0.00 -> 8.40 mm
- net hv-1: track 6.20 -> 0.00 mm
- net _5v_reg-vcc: track 0.00 -> 6.20 mm
- net _5v_reg.ic-l1: track 0.00 -> 2.59 mm
- net _3v3_reg.ic-l1: track 0.00 -> 2.59 mm
- net _5v_reg.ic-l2: track 0.00 -> 2.54 mm
- net _3v3_reg.ic-l2: track 0.00 -> 2.54 mm
- net out: track 2.08 -> 0.00 mm
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
Commit message: Remove stray net
Connections:
- U3 pad 7: _7 -> (no net)
Changed lines of the file:
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@@
     (net 60 "cathode")
     (net 61 "led_dout")
-    (net 63 "_7")
     (footprint "atopile:C0402-b3ef17"
         (layer "F.Cu")
@@
             (remove_unused_layers no)
             (pintype "stereo")
-            (net 63 "_7"))
+            (net 0 ""))
         (pad "8" smd rect
             (at 1.27 -2 90)
